File: onboard-circuit/onboard-circuit.kicad_sch (KiCad schematic)
At the start: 11 parts, among them J1 Conn_01x15, K1 SIEMENS

Commit message: labels, datasheet, circuit doku
Parts:
- removed J1: Conn_01x15, symbol Connector_Generic:Conn_01x15
- added J2: Edge Connector, symbol Connector:Conn_01x15_Pin
Connections:
- net +24V: now also J2.3 (Pin_3), J2.4 (Pin_4)
- net GND: now also J2.1 (Pin_1), J2.2 (Pin_2)
- net at C.2, M.2 (-), R10.2: now also J2.15 (Pin_15)
- net at K1.11: now also J2.14 (Pin_14)
- net at D9.1 (K): now also J2.13 (Pin_13)
Other:
- moved on the sheet: D8, GRAYCODE-LIGHT, R7

Commit message: completed onboard circuit
Parts:
- added D1, D2, D3, D4, D5, D6, D7: D, symbol Device:D
- added D1, D11, D13, D15, D2, D4, D6: D_Photo, symbol Device:D_Photo
- added Q1, Q2, Q3, Q4, Q5, Q6, Q7: NPN, symbol Simulation_SPICE:NPN
- added R1, R2, R3, R4, R5, R6, R8: 6K8, symbol Device:R
- renumbered GRAYCODE-LIGHT to D
Connections:
- net GND: now also Q1.3 (E), Q2.3 (E), Q3.3 (E), Q4.3 (E), Q5.3 (E), Q6.3 (E), Q7.3 (E), R1.2, R2.2, R3.2, R4.2, R5.2, R6.2, R8.2
- net at J2.10 (Pin_10): now also D11.1 (K), D3.2 (A)
- net at J2.11 (Pin_11): now also D13.1 (K), D2.2 (A)
- net at J2.12 (Pin_12): now also D1.2 (A), D15.1 (K)
- net at J2.6 (Pin_6): now also D1.1 (K), D7.2 (A)
- net at J2.7 (Pin_7): now also D2.1 (K), D6.2 (A)
- net at J2.8 (Pin_8): now also D4.1 (K), D5.2 (A)
- net at J2.9 (Pin_9): now also D4.2 (A), D6.1 (K)
- new net: D2.1 (K), Q6.1 (C)
- new net: D13.2 (A), Q6.2 (B), R2.1
- new net: D2.2 (A), Q2.2 (B), R6.1
- new net: D11.2 (A), Q5.2 (B), R3.1
- new net: D1.1 (K), Q7.1 (C)
- new net: D3.1 (K), Q5.1 (C)
- new net: D6.2 (A), Q4.2 (B), R4.1
- new net: D7.1 (K), Q1.1 (C)
- new net: D1.2 (A), Q1.2 (B), R8.1
- new net: D4.1 (K), Q4.1 (C)
- new net: D5.1 (K), Q3.1 (C)
- new net: D6.1 (K), Q2.1 (C)
- new net: D15.2 (A), Q7.2 (B), R1.1
- new net: D4.2 (A), Q3.2 (B), R5.1
Other:
- note added: "GRAYCODE LIGHT"
- note added: "GRAYCODE SENSORS"
- note added: "Q1 ... Q7 are in CA3081 7 Channel Common Emitter NPN Array"
- moved on the sheet: C, C1, D8, D9, J2, K1, M, R10, R7, R9
