File: pcb/plug-module/plug-module.kicad_sch (KiCad schematic)
At the start: 37 parts, among them J1 Conn_01x10_Pin, J10 Conn_01x01_Pin, J11 Conn_01x01_Pin, J12 Conn_01x01_Pin, J2 Conn_01x04_Pin, J3 Conn_01x15_Socket, J4 Conn_01x04_Pin, J5 Conn_01x10_Pin, J6 Conn_01x01_Pin, J7 Conn_01x01_Pin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

Commit message: r net 100k
Parts:
- RN1: value 390K -> 100K
Changed lines of the file:
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@@
 			)
 		)
-		(property "Value" "390K"
+		(property "Value" "100K"
 			(at 57.912 64.9661 0)
 			(effects
